File: eda/eda.kicad_pcb (KiCad board)
At the start: 2 copper layers, 44 x 72 mm, 86 parts, among them J1 SJ-3523-SMT-TR, J2 SJ-3523-SMT-TR, J3 FTSH-105-01-L-DV-K-A-P-TR, J4 AYF531035, Q1 DMP2045U-7, SW1 KMR221NG LFS, SW2 KMR221NG LFS, SW3 KMR221NG LFS, SW4 KMR221NG LFS, U1 MCP6042T-I/MS, U2 STM32U083KCU6, Y1 32.768kHz 7pF

Commit message: updates
Parts:
- C17: moved to F.Cu
- moved FID4 54.3 mm to (112.2, 153.0)
- moved SW3 43.6 mm to (141.4, 121.5), turned to -90 degrees
- moved R3 36.1 mm to (139.5, 155.0)
- moved R14 35.0 mm to (129.3, 148.4)
- moved R15 33.7 mm to (129.3, 149.9)
- moved C4 31.3 mm to (129.5, 146.1), turned to -90 degrees
- moved C5 31.2 mm to (128.0, 146.1), turned to 90 degrees
- moved R13 31.0 mm to (130.9, 146.1), turned to -90 degrees
- moved FID1 30.4 mm to (103.0, 107.5)
- moved R4 28.5 mm to (135.5, 155.0), turned to 180 degrees
- moved FID2 21.6 mm to (142.6, 154.4)
- moved C18 3.28 mm to (133.8, 137.0)
- moved C17 3.18 mm to (136.5, 138.9)
- moved C14 0.50 mm to (138.8, 137.6)
Routing:
- net VBAT: track 5.40 -> 147.6 mm, vias 0 -> 15
- net AUDIO_R_IN: track 0.00 -> 141.1 mm, vias 0 -> 6
- net AUDIO_L_IN: track 0.00 -> 97.0 mm, vias 0 -> 3
- net SWDIO: track 0.00 -> 49.6 mm, vias 0 -> 3
- net SWCLK: track 0.00 -> 47.0 mm, vias 0 -> 3
- net ENV_OUT: track 0.00 -> 44.7 mm, vias 0 -> 2
- net NRST: track 0.00 -> 41.0 mm, vias 0 -> 3
- net MUSIC_PRESENT: track 2.08 -> 37.5 mm, vias 0 -> 3
- net BTN_SELECT: track 0.00 -> 33.8 mm
- net UART_RX: track 0.00 -> 28.8 mm, vias 0 -> 2
- net AUDIO_VMID: track 8.50 -> 35.8 mm, vias 0 -> 1
- net BTN_DANCE_A: track 0.00 -> 27.1 mm
- net POWER.VBAT_CELL: track 0.00 -> 26.2 mm, vias 0 -> 2
- net BOOT0: track 0.00 -> 25.8 mm, vias 0 -> 3
- net UART_TX: track 0.00 -> 24.1 mm, vias 0 -> 2
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- added copper zone on B.Cu, net GND

Commit message: new changes
Parts:
- J3: footprint lena_registry_components_Samtec_FTSH-105-01-L-DV-K-A-P-TR@0.1.0:FTSH-105-01-L-DV-K-A-P-TR -> lena_registry_components_Samtec_FTSH-105-01-L-DV-K-A-P-TR@0.1.1:FTSH-105-01-L-DV-K-A-P-TR
Routing:
- net GND: track 18.9 -> 26.2 mm, vias 37 -> 41
- net VBAT: track 147.6 -> 144.7 mm
- net MCU.OSC32_OUT: track 7.20 -> 6.48 mm
- net MCU.OSC32_IN: track 7.54 -> 6.81 mm
- net NRST: track 41.0 -> 40.3 mm
