File: eda/eda.kicad_sch (KiCad schematic)
At the start: 86 parts, among them J1 SJ-3523-SMT-TR, J2 SJ-3523-SMT-TR, J3 FTSH-105-01-L-DV-K-A-P-TR, J4 AYF531035, Q1 DMP2045U-7, SW1 KMR221NG LFS, SW2 KMR221NG LFS, SW3 KMR221NG LFS, SW4 KMR221NG LFS, U1 MCP6042T-I/MS, U2 STM32U083KCU6, Y1 32.768kHz 7pF

Commit message: new changes
Other:
- note removed: "10-pin Cortex SWD header and probe pads. Probe VTref only senses VBAT."
- note removed: "AUDIO PASSTHROUGH"
- note removed: "AUDIO SENSE"
- note removed: "CR2032 cell, reverse-polarity P-FET, >=100 uF bulk. No regulator: everything runs from VBAT."
- note removed: "DEBUG"
- note removed: "DISPLAY"
- note removed: "Fully passive stereo path, jack to jack. Works with a dead cell or MCU in reset."
- note removed: "HMI"
- note removed: "M2 mounting holes and fiducials."
- note removed: "MCU"
- note removed: "MECHANICAL"
- note removed: "Non-loading 100k tap, precision half-wave envelope detector (U1A), music-present comparator (U1B). Option B direct-ADC parts are DNP."
- note removed: "POWER"
- note removed: "STM32U083KCU6, decoupling, 32.768 kHz LSE, BOOT0 pull-down, NRST filter."
- note removed: "Select, Dance A, Dance B (internal pull-ups) and the pinhole reset switch."
- note removed: "Sharp LS013B7DH03 memory LCD on 10-pin 0.5 mm FPC (J4). EXTMODE strap selects EXTCOMIN mode."
- title: funbit: Sony PET-F7 Funbbit recreation -> (none)
- moved on the sheet: BT1, C1, C10, C11, C12, C13, C14, C15, C16, C17, C18, C19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
